File: HPA4.kicad_sch (KiCad schematic)
At the start: 188 parts, among them J10 PWR L, J11 LIN, J12 Conn_01x01_Male, J13 Servo, J2 RIN, J3 Conn_01x01_Male, J4 PWR R, J5 Servo, J6 ROUT, J7 LOUT, J8 RELAY PWR, J9 LED, K1 G6H-2, Q1 BC560C, Q10 BC560C, Q11 TTA004B, Q12 BC550C, Q13 TTC004B, Q14 BC560C, Q15 TTA004B, Q16 BC550C, Q17 TTC004B, Q18 KSC1845, Q19 BC550C, Q2 BC560C, Q20 BC550C, Q21 BC550C, Q22 BC550C, Q23 MMBT3906, Q24 MMBT3906, Q25 MMBT3906, Q26 MMBT3904, Q27 BC560C, Q28 BC560C, Q29 BC560C, Q3 BC560C, Q30 BC560C, Q31 KSA992, Q32 BC560C, Q33 TTA004B, Q34 TTC004B, Q35 BC550C, Q36 BC560C, Q37 TTA004B, Q38 TTC004B, Q39 BC550C, Q4 BC560C, Q40 BC560C, Q41 TTA004B, Q42 BC550C, Q43 TTC004B, Q44 KSC1845, Q45 BC550C, Q46 BC550C, Q47 BC550C, Q48 BC550C, Q5 KSA992, Q6 BC560C, Q7 TTA004B, Q8 TTC004B, Q9 BC550C, U1 LT1761-BYP, U2 LT1964-BYP, U3 OPA604, U4 LM555, U5 LT1761-BYP, U6 LT1964-BYP, U7 OPA604

Commit message: Corrected some incorrect resistor values in the left channel to match prior revisions to right channel.
Parts:
- R44, R73: value 100 -> 221
- R54, R65: value 22 -> 100
- R55, R64: value 12 -> 90.9
- R58: value 5.6K -> 30K
- R76: value 750 -> 1500
- R77: value 332 -> 750
Changed lines of the file:
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@@
 			)
 		)
-		(property "Value" "22"
+		(property "Value" "100"
 			(at 180.34 381.635 90)
 			(effects
@@
 			)
 		)
-		(property "Value" "100"
+		(property "Value" "221"
 			(at 205.613 325.12 90)
 			(effects
@@
 			)
 		)
-		(property "Value" "12"
+		(property "Value" "90.9"
 			(at 205.74 389.255 90)
 			(effects
@@
 			)
 		)
-		(property "Value" "12"
+		(property "Value" "90.9"
 			(at 205.74 411.48 90)
 			(effects
@@
 			)
 		)
-		(property "Value" "100"
+		(property "Value" "221"
 			(at 205.613 472.44 90)
 			(effects
@@
 			)
 		)
-		(property "Value" "5.6K"
+		(property "Value" "30K"
 			(at 161.29 400.685 90)
 			(effects
@@
 			)
 		)
-		(property "Value" "332"
+		(property "Value" "750"
 			(at 303.403 509.143 0)
 			(effects
@@
 			)
 		)
-		(property "Value" "22"
+		(property "Value" "100"
 			(at 180.34 418.465 90)
 			(effects
@@
 			)
 		)
-		(property "Value" "750"
+		(property "Value" "1500"
 			(at 314.96 499.11 90)
 			(effects
